Commit message: add readme and adjust some params

File: urdf/sensor_pod.urdf (robot description, URDF)
Before this commit: robot cartographer_sensor_pod, 3 links, 2 joints
Links:
- added link camera0_link; visual box size=0.02 0.01 0.02
Joints:
- added joint camera0_link_joint: type fixed, parent base_link, child camera0_link, origin xyz=0.0 0.0 0.0 rpy=0.0 0.0 0
